Commit message: Fix laser sensor frame and joint configuration
Removed unused IMU and camera macros, added laser components.

File: fishbot_description/urdf/fishbot/sensor/laser.urdf.xacro (robot description, xacro)
@@ -1,100 +1,66 @@
 <?xml version="1.0"?>
 <robot xmlns:xacro="http://www.ros.org/wiki/xacro">
-<xacro:include filename="$(find fishbot_description)/urdf/fishbot/common_inertia.xacro"/>
-  <xacro:macro name="imu_xacro" params="xyz">
-    <link name="imu_link">
-      <visual>
-        <origin xyz="0.0 0.0 0.0" rpy="0.0 0.0 0.0"/>
-        <geometry>
-          <box size="0.02 0.02 0.02"/>
-        </geometry>
-        <material name="black">
-          <color rgba="0.0 0.0 0.0 0.5"/>
-        </material>
-      </visual>
-    </link>
-    <joint name="imu_joint" type="fixed">
-      <parent link="base_link"/>
-      <child link="imu_link"/>
-      <origin xyz="${xyz}" rpy="0.0 0.0 0.0"/>
-    </joint>
-  </xacro:macro>
-  <xacro:macro name="camera_xacro" params="xyz">
-    <link name="camera_link">
-      <visual>
-        <origin xyz="0.0 0.0 0.0" rpy="0.0 0.0 0.0"/>
-        <geometry>
-          <box size="0.02 0.02 0.02"/>
-        </geometry>
-        <material name="black">
-          <color rgba="0.0 0.0 0.0 0.5"/>
-        </material>
-      </visual>
-    </link>
-    <joint name="camera_joint" type="fixed">
-      <parent link="base_link"/>
-      <child link="camera_link"/>
-      <origin xyz="${xyz}" rpy="0.0 0.0 0.0"/>
-    </joint>
-  </xacro:macro>
-  <xacro:macro name="laser_xacro" params="xyz">
-    <link name="laser_cylinder_link">
-      <visual>
-        <origin xyz="0.0 0.0 0.0" rpy="0.0 0.0 0.0"/>
-        <geometry>
-          <cylinder radius="0.01" length="0.10"/>
-        </geometry>
-        <material name="black">
-          <color rgba="0.0 0.0 0.0 1.0"/>
-        </material>
-      </visual>
-      <collision>
-        <origin xyz="0.0 0.0 0.0" rpy="0.0 0.0 0.0"/>
-        <geometry>
-          <cylinder radius="0.01" length="0.10"/>
-        </geometry>
-        <material name="black">
-          <color rgba="0.0 0.0 0.0 1.0"/>
-        </material>
-      </collision>
-      <xacro:cylinder_inertia m="0.05" r="0.01" h="0.10" />
-    </link>
-    <link name="laser_link">
-      <visual>
-        <origin xyz="0.0 0.0 0.0" rpy="0.0 0.0 0.0"/>
-        <geometry>
-          <cylinder radius="0.02" length="0.02"/>
-        </geometry>
-        <material name="black">
-          <color rgba="0.0 0.0 0.0 1.0"/>
-        </material>
-      </visual>
-      <collision>
-        <origin xyz="0.0 0.0 0.0" rpy="0.0 0.0 0.0"/>
-        <geometry>
-          <cylinder radius="0.02" length="0.02"/>
-        </geometry>
-        <material name="black">
-          <color rgba="0.0 0.0 0.0 1.0"/>
-        </material>
-      </collision>
-      <xacro:cylinder_inertia m="0.10" r="0.02" h="0.02" />
-    </link>
-    <joint name="laser_joint" type="fixed">
-      <parent link="laser_cylinder_link"/>
-      <child link="laser_link"/>
-      <origin xyz="0.0 0.0 0.05" rpy="0.0 0.0 0.0"/>
-    </joint>
-    <joint name="laser_cylinder_joint" type="fixed">
-      <parent link="base_link"/>
-      <child link="laser_cylinder_link"/>
-      <origin xyz="${xyz}" rpy="0.0 0.0 0.0"/>
-    </joint>
-    <gazebo reference="laser_cylinder_link">
-      <material>Gazebo/Black</material>
-    </gazebo>
-    <gazebo reference="laser_link">
-        <material>Gazebo/Black</material>
-    </gazebo>
-  </xacro:macro>
+   <xacro:include filename="$(find fishbot_description)/urdf/fishbot/common_inertia.xacro" />
+    <xacro:macro name="laser_xacro" params="xyz">
+        <gazebo reference="laser_cylinder_link">
+            <material>Gazebo/Black</material>
+        </gazebo>
+        <gazebo reference="laser_link">
+            <material>Gazebo/Black</material>
+        </gazebo>
+        <!-- ============雷达支撑杆================ -->
+        <link name="laser_cylinder_link">
+            <visual>
+                <origin xyz="0.0 0.0 0.0" rpy="0.0 0.0 0.0" />
+                <geometry>
+                    <cylinder length="0.10" radius="0.01" />
+                </geometry>
+                <material name="black">
+                    <color rgba="0.0 0.0 0.0 1.0" />
+                </material>
+            </visual>
+            <collision>
+                <origin xyz="0.0 0.0 0.0" rpy="0.0 0.0 0.0" />
+                <geometry>
+                    <cylinder length="0.10" radius="0.01" />
+                </geometry>
+                <material name="black">
+                    <color rgba="0.0 0.0 0.0 1.0" />
+                </material>
+            </collision>
+            <xacro:cylinder_inertia m="0.05" r="0.01" h="0.10" />
+        </link>
+        <joint name="laser_cylinder_joint" type="fixed">
+            <parent link="base_link" />
+            <child link="laser_cylinder_link" />
+            <origin xyz="${xyz}" />
+        </joint>
+        <!-- ============雷达================ -->
+        <link name="laser_link">
+            <visual>
+                <origin xyz="0.0 0.0 0.0" rpy="0.0 0.0 0.0" />
+                <geometry>
+                    <cylinder length="0.02" radius="0.02" />
+                </geometry>
+                <material name="black">
+                    <color rgba="0.0 0.0 0.0 1.0" />
+                </material>
+            </visual>
+            <collision>
+                <origin xyz="0.0 0.0 0.0" rpy="0.0 0.0 0.0" />
+                <geometry>
+                    <cylinder length="0.02" radius="0.02" />
+                </geometry>
+                <material name="black">
+                    <color rgba="0.0 0.0 0.0 1.0" />
+                </material>
+            </collision>
+            <xacro:cylinder_inertia m="0.10" r="0.02" h="0.02" />
+        </link>
+        <joint name="laser_joint" type="fixed">
+            <parent link="laser_cylinder_link" />
+            <child link="laser_link" />
+            <origin xyz="0 0 0.05" />
+        </joint>
+    </xacro:macro>
 </robot>
